Commit message: sensors

File: src/robot/urdf/rover.urdf (robot description, URDF)
Before this commit: robot rover, 18 links, 17 joints
Links:
- added link camera_link
- added link lidar_link
Joints:
- added joint camera_link_joint: type fixed, parent Base_link, child camera_link, origin xyz=0.10 0.0 0.05 rpy=-1.57060 -1.57057 0
- added joint lidar_joint: type fixed, parent Base_link, child lidar_link, origin xyz=0.0 0.0 0.15 rpy=0 0 0
